File: ev-2027-wiring/ev-2027-wiring.kicad_sch (KiCad schematic)
At the start: 16 parts, among them SW1 SW_DIP_x01, U1 SN74LVC2G17DBV

Commit message: fix all electrical circuits
Parts:
- renumbered C3 to CS2
Connections:
- net at CS3.BL (Blacklight): now also CS1.7
- no-connect marks 0 -> 45
Other:
- title: (none) -> CVHS EV 2026-2027 Vehicle Wiring Schematic
- moved on the sheet: D1
