File: ev-2027-wiring/.history/ev-2027-wiring.kicad_pcb (KiCad board)
At the start: 2 copper layers, 16 parts, among them SW1 SW_DIP_x01, U1 SN74LVC2G17DBV

Commit message: pcb placement
Parts:
- moved P3 43.2 mm to (149.4, 53.4)
- moved CS5 35.3 mm to (84.8, 74.3)
- moved CS1 15.5 mm to (120.8, 75.2), turned to -90 degrees
- moved CS4 9.08 mm to (129.2, 123.5)

Commit message: pbc changes
Parts:
- moved C2 109.8 mm to (57.5, 80.0)
- moved CS4 97.0 mm to (52.9, 63.6)
- moved M2 86.2 mm to (45.5, 48.5), turned to 90 degrees
- moved U1 78.1 mm to (50.6, 81.0)
- moved CS5 72.7 mm to (157.5, 72.0)
- moved C1 70.8 mm to (66.5, 56.5)
- moved D1 68.9 mm to (110.4, 48.0)
- moved M1 65.8 mm to (154.0, 55.5)
- moved P1 54.8 mm to (196.5, 78.7)
- moved P2 46.9 mm to (111.9, 126.2)
- moved P3 41.5 mm to (107.9, 53.4)
- moved F1 35.4 mm to (185.1, 115.5)
- moved CS2 29.0 mm to (117.0, 85.9)
- moved CS1 26.4 mm to (94.4, 75.7)
- moved SW1 18.4 mm to (94.0, 125.5)
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Changed lines of the file:
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@@
 	(footprint "Teensy:Pololu_DRV8874_4035"
 		(layer "F.Cu")
-		(at 129.185 123.5)
+		(at 52.85 63.58)
 		(descr "Pololu DRV8874 carrier #4035 (md41a), 15.2x17.8mm, 2x7 0.1in rows 0.5in apart, TOP VIEW chip-side up. Pin order verified against Pololu labeled pinout photo; pads named to match EV_2027:DRV8874_Carrier.")
 		(tags "Pololu_DRV8874_4035")
@@
 	(footprint "Teensy:Teensy41_PinNames"
 		(layer "F.Cu")
-		(at 120.8184 75.24 -90)
+		(at 94.38 75.65 -90)
 		(property "Reference" "CS1"
 			(at 0 -10.16 90)
@@
 	(footprint "Teensy:NEMA8_Stepper_JST_XH_1x04"
 		(layer "F.Cu")
-		(at 152.895 121.335)
+		(at 154 55.5)
 		(descr "4-pin JST-XH for the Pololu #1204 NEMA 8 stepper. Order: A (A1 black), C (A2 green), B (B1 red), D (B2 blue), so each coil pair is adjacent; matches EV:Pololu_#1204 symbol. Based on KiCad JST XH series connector, B4B-XH-A (http://www.jst-mfg.com/product/pdf/eng/eXH.pdf)")
 		(tags "connector JST XH vertical")
@@
 	(footprint "Teensy:Reg8V_ScrewTerminal_1x04_P5.08mm"
 		(layer "F.Cu")
-		(at 143.685 91.665)
+		(at 111.88 126.1725)
 		(descr "4-pin 5.08mm screw terminal for an off-board 8V regulator module: VIN, GND, VOUT, EN, matching EV:8V_Voltage_Regulator_Placeholder. Based on KiCad Terminal Block Phoenix MKDS-1,5-4-5.08, 4 pins, pitch 5.08mm, size 20.3x9.8mm, drill diameter 1.3mm, pad diameter 2.6mm, http://www.farnell.com/datasheets/100425.pdf")
 		(tags "THT Terminal Block Phoenix MKDS-1,5-4-5.08 pitch 5.08mm size 20.3x9.8mm drill 1.3mm pad 2.6mm")
@@
 	(footprint "Diode_THT:D_DO-35_SOD27_P7.62mm_Horizontal"
 		(layer "F.Cu")
-		(at 110.165 116.925)
+		(at 110.38 48)
 		(descr "Diode, DO-35_SOD27 series, Axial, Horizontal, pin pitch=7.62mm, length*diameter=4*2mm^2, http://www.diodes.com/_files/packages/DO-35.pdf")
 		(tags "Diode DO-35_SOD27 series Axial Horizontal pin pitch 7.62mm  length 4mm diameter 2mm")
@@
 	(footprint "Capacitor_SMD:C_0805_2012Metric"
 		(layer "F.Cu")
-		(at 163.865 107.345)
+		(at 57.5 80)
 		(descr "Capacitor SMD 0805 (2012 Metric), square (rectangular) end terminal, IPC-7351 nominal, (Body size source: IPC-SM-782 page 76, https://www.pcb-3d.com/wordpress/wp-content/uploads/ipc-sm-782a_amendment_1_and_2.pdf, https://docs.google.com/spreadsheets/d/1BsfQQcO9C6DZCsRaXUlFlo91Tg2WpOkGARC1WS5S8t0/edit?usp=sharing)")
 		(tags "capacitor")
@@
 	(footprint "Button_Switch_SMD:SW_SPST_CK_KMS2xxGP"
 		(layer "F.Cu")
-		(at 111.865 121.175)
+		(at 94 125.5)
 		(descr "Microminiature SMT Side Actuated, 4.2 x 2.8 x 1.42mm with pegs, https://www.ckswitches.com/media/1482/kms.pdf")
 		(tags "Switch SPST KMS2")
@@
 	(footprint "Capacitor_THT:CP_Radial_D6.3mm_P2.50mm"
 		(layer "F.Cu")
-		(at 111.400241 111.225)
+		(at 66.5 56.5)
 		(descr "CP, Radial series, Radial, pin pitch=2.50mm, diameter=6.3mm, height=7mm, Electrolytic Capacitor")
 		(tags "CP Radial series Radial pin pitch 2.50mm diameter 6.3mm height 7mm Electrolytic Capacitor")
@@
 	(footprint "Teensy:Pololu_DRV8834_2134"
 		(layer "F.Cu")
-		(at 84.85 74.35)
+		(at 157.5 72)
 		(descr "Pololu DRV8834 carrier #2134 (md22a), 15.2x20.3mm, 2x8 0.1in rows 0.5in apart, TOP VIEW chip-side up (pot at the DIR/GND end). Pin order verified against Pololu wiring diagram; pads named to match EV_2027:DRV8834_Carrier. CONFIG/VREF are optional jumper pins, unused.")
 		(tags "Pololu_DRV8834_2134")
@@
 	(footprint "Teensy:Pololu_25D_Motor_Encoder_Header_1x06"
 		(layer "F.Cu")
-		(at 106.295 109.595)
+		(at 45.46 48.5 90)
 		(descr "1x6 0.1in male header for the Pololu 25D gearmotor encoder cable. Pin order Red (M1), Black (M2), Green (enc GND), Blue (enc Vcc), Yellow (A), White (B), matching EV:Pololu_#4801. Verify against your cable before soldering. Based on KiCad Through hole straight pin header, 1x06, 2.54mm pitch, single row")
 		(tags "Through hole pin header THT 1x06 2.54mm single row")
 		(property "Reference" "M2"
-			(at 0 -2.38 0)
+			(at 0 -2.38 90)
 			(layer "F.SilkS")
 			(effects
@@
 		)
 		(property "Value" "~"
-			(at 0 15.08 0)
+			(at 0 15.08 90)
 			(layer "F.Fab")
 			(effects
@@
 		)
 		(property "Datasheet" ""
-			(at 0 0 0)
+			(at 0 0 90)
 			(layer "F.Fab")
 			(hide yes)
@@
 		)
 		(property "Description" ""
-			(at 0 0 0)
+			(at 0 0 90)
 			(layer "F.Fab")
 			(hide yes)
@@
 		)
 		(property "KiLib_Generator" "connector/pin_header_socket"
-			(at 0 0 0)
+			(at 0 0 90)
 			(layer "F.SilkS")
 			(hide yes)
@@
 		)
 		(fp_line
-			(start -1.38 1.27)
-			(end -1.38 14.08)
+			(start 1.38 1.27)
+			(end 1.38 14.08)
 			(stroke
 				(width 0.12)
@@
 		)
 		(fp_line
-			(start -1.38 14.08)
-			(end 1.38 14.08)
+			(start -1.38 1.27)
+			(end -1.38 14.08)
 			(stroke
 				(width 0.12)
@@
 		)
 		(fp_line
-			(start 1.38 1.27)
+			(start -1.38 14.08)
 			(end 1.38 14.08)
 			(stroke
@@
 		)
 		(fp_line
-			(start -1.27 -0.635)
-			(end -0.635 -1.27)
+			(start 1.27 -1.27)
+			(end 1.27 13.97)
 			(stroke
 				(width 0.1)
@@
 		)
 		(fp_line
-			(start -1.27 13.97)
-			(end -1.27 -0.635)
+			(start -0.635 -1.27)
+			(end 1.27 -1.27)
 			(stroke
 				(width 0.1)
@@
 		)
 		(fp_line
-			(start -0.635 -1.27)
-			(end 1.27 -1.27)
+			(start -1.27 -0.635)
+			(end -0.635 -1.27)
 			(stroke
 				(width 0.1)
@@
 		)
 		(fp_line
-			(start 1.27 -1.27)
-			(end 1.27 13.97)
+			(start 1.27 13.97)
+			(end -1.27 13.97)
 			(stroke
 				(width 0.1)
@@
 		)
 		(fp_line
-			(start 1.27 13.97)
-			(end -1.27 13.97)
+			(start -1.27 13.97)
+			(end -1.27 -0.635)
 			(stroke
 				(width 0.1)
@@
 		)
 		(fp_text user "${REFERENCE}"
-			(at 0 6.35 90)
+			(at 0 6.35 0)
 			(layer "F.Fab")
 			(effects
@@
 		)
 		(pad "Black" thru_hole circle
-			(at 0 2.54)
+			(at 0 2.54 90)
 			(size 1.7 1.7)
 			(drill 1)
@@
 		)
 		(pad "Blue" thru_hole circle
-			(at 0 7.62)
+			(at 0 7.62 90)
 			(size 1.7 1.7)
 			(drill 1)
@@
 		)
 		(pad "Green" thru_hole circle
-			(at 0 5.08)
+			(at 0 5.08 90)
 			(size 1.7 1.7)
 			(drill 1)
@@
 		)
 		(pad "Red" thru_hole rect
-			(at 0 0)
+			(at 0 0 90)
 			(size 1.7 1.7)
 			(drill 1)
@@
 		)
 		(pad "White" thru_hole circle
-			(at 0 12.7)
+			(at 0 12.7 90)
 			(size 1.7 1.7)
 			(drill 1)
@@
 		)
 		(pad "Yellow" thru_hole circle
-			(at 0 10.16)
+			(at 0 10.16 90)
 			(size 1.7 1.7)
 			(drill 1)
@@
 	(footprint "Teensy:Battery_ScrewTerminal_1x02_P5.08mm"
 		(layer "F.Cu")
-		(at 152.985 112.075)
+		(at 196.455 78.6725)
 		(descr "2-pin 5.08mm screw terminal for the 8xAA battery pack. Pads VOUT (pack +) and GND, matching the EV:Battery_Pack symbol. Based on KiCad Terminal Block Phoenix MKDS-1,5-2-5.08, 2 pins, pitch 5.08mm, size 10.2x9.8mm, drill diameter 1.3mm, pad diameter 2.6mm, http://www.farnell.com/datasheets/100425.pdf")
 		(tags "THT Terminal Block Phoenix MKDS-1,5-2-5.08 pitch 5.08mm size 10.2x9.8mm drill 1.3mm pad 2.6mm")
@@
 	(footprint "Teensy:GY-BNO08X_1x10_P2.54mm"
 		(layer "F.Cu")
-		(at 142.445 99.875)
+		(at 117 85.88)
 		(descr "GY-BNO08X (BNO080/BNO085/BNO086) IMU module, single 1x10 0.1in header, TOP VIEW: VCC at pin 1 (top) down to PS0 (bottom). Pads named by the module silkscreen labels. Board outline not included: module size varies by seller, measure yours.")
 		(tags "BNO085 BNO08X GY IMU 1x10")
@@
 	(footprint "Package_TO_SOT_SMD:SOT-23-6"
 		(layer "F.Cu")
-		(at 117.715 121.1)
+		(at 50.6375 81.05)
 		(descr "SOT, 6 Pin (JEDEC MO-178 Var AB https://www.jedec.org/document_search?search_api_views_fulltext=MO-178)")
 		(tags "SOT TO_SOT_SMD")
@@
 	(footprint "Fuse:Fuseholder_Blade_Mini_Keystone_3568"
 		(layer "F.Cu")
-		(at 153.235 99.995)
+		(at 185.08 115.5)
 		(descr "fuse holder, car blade fuse mini, http://www.keyelco.com/product-pdf.cfm?p=306")
 		(tags "car blade fuse mini")
@@
 	(footprint "Teensy:Display_ST7789_Header_1x08_P2.54mm_Named"
 		(layer "F.Cu")
-		(at 147.095 99.875)
+		(at 150 90.92)
 		(descr "8-pin 0.1in male header for Waveshare 1.69in ST7789V2 display on jumper wires. Order matches the display cable: VCC GND DIN CLK CS DC RST BL (pin 1 = VCC, square pad). Pads named by signal to match symbols that use pin names; use PinHeader_1x08_P2.54mm_Vertical for symbols numbered 1-8.")
 		(tags "header 1x08 display ST7789 jumper")
@@
 	(footprint "Teensy:Pololu_D24V22F5_2858"
 		(layer "F.Cu")
-		(at 149.38 53.38)
+		(at 107.88 53.38)
 		(descr "Pololu D24V22F5 5V regulator #2858 (reg19a), 17.8x17.8mm, TOP VIEW. Main row PG/EN/VIN/GND/VOUT plus extra GND; two 2.18mm mounting holes. Verified vs Pololu labeled pinout photo and dimension drawing. Pads numbered to match EV_2027:D24V22F5 (VIN=1 GND=2 VOUT=3 EN=4).")
 		(tags "Pololu_D24V22F5_2858")
