File: ev-2027-wiring/.history/ev-2027-wiring.kicad_sch (KiCad schematic)
At the start: 16 parts, among them SW1 SW_DIP_x01, U1 SN74LVC2G17DBV

Commit message: assigned footprints and inserted into pcb
errors still exist
Parts:
- C1: footprint (none) -> Capacitor_THT:CP_Radial_D6.3mm_P2.50mm
- C2: footprint (none) -> Capacitor_SMD:C_0805_2012Metric
- CS1: footprint (none) -> Teensy:Teensy41_PinNames
- CS2: footprint (none) -> Teensy:GY-BNO08X_1x10_P2.54mm
- CS3: footprint (none) -> Teensy:Display_ST7789_Header_1x08_P2.54mm_Named
- CS4: footprint (none) -> Teensy:Pololu_DRV8874_4035
- CS5: footprint (none) -> Teensy:Pololu_DRV8834_2134
- F1: footprint Package_LCC:PLCC-84_29.3x29.3mm_P1.27mm -> Fuse:Fuseholder_Blade_Mini_Keystone_3568
- M1: footprint (none) -> Teensy:NEMA8_Stepper_JST_XH_1x04
- M2: footprint (none) -> Teensy:Pololu_25D_Motor_Encoder_Header_1x06
- P1: footprint (none) -> Teensy:Battery_ScrewTerminal_1x02_P5.08mm
- P2: footprint (none) -> Teensy:Reg8V_ScrewTerminal_1x04_P5.08mm
- P3: footprint (none) -> Teensy:Pololu_D24V22F5_2858
Changed lines of the file:
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@@
 			)
 		)
-		(property "Footprint" ""
+		(property "Footprint" "Teensy:Battery_ScrewTerminal_1x02_P5.08mm"
 			(at 83.82 50.8 0)
 			(hide yes)
@@
 			)
 		)
-		(property "Footprint" "Package_LCC:PLCC-84_29.3x29.3mm_P1.27mm"
+		(property "Footprint" "Fuse:Fuseholder_Blade_Mini_Keystone_3568"
 			(at 104.14 31.75 0)
 			(hide yes)
@@
 			)
 		)
-		(property "Footprint" ""
+		(property "Footprint" "Teensy:Display_ST7789_Header_1x08_P2.54mm_Named"
 			(at 66.04 77.47 0)
 			(hide yes)
@@
 			)
 		)
-		(property "Footprint" ""
+		(property "Footprint" "Capacitor_SMD:C_0805_2012Metric"
 			(at 223.52 123.19 0)
 			(hide yes)
@@
 			)
 		)
-		(property "Footprint" ""
+		(property "Footprint" "Teensy:Pololu_25D_Motor_Encoder_Header_1x06"
 			(at 270.51 123.19 0)
 			(hide yes)
@@
 			)
 		)
-		(property "Footprint" ""
+		(property "Footprint" "Capacitor_THT:CP_Radial_D6.3mm_P2.50mm"
 			(at 234.95 58.42 0)
 			(hide yes)
@@
 			)
 		)
-		(property "Footprint" ""
+		(property "Footprint" "Teensy:Pololu_D24V22F5_2858"
 			(at 175.26 44.45 0)
 			(hide yes)
@@
 			)
 		)
-		(property "Footprint" ""
+		(property "Footprint" "Teensy:Pololu_DRV8874_4035"
 			(at 208.28 118.11 0)
 			(hide yes)
@@
 			)
 		)
-		(property "Footprint" ""
+		(property "Footprint" "Teensy:Reg8V_ScrewTerminal_1x04_P5.08mm"
 			(at 217.17 36.83 0)
 			(hide yes)
@@
 			)
 		)
-		(property "Footprint" ""
+		(property "Footprint" "Teensy:Pololu_DRV8834_2134"
 			(at 205.74 83.82 0)
 			(hide yes)
@@
 			)
 		)
-		(property "Footprint" ""
+		(property "Footprint" "Teensy:NEMA8_Stepper_JST_XH_1x04"
 			(at 273.05 63.5 0)
 			(hide yes)
@@
 			)
 		)
-		(property "Footprint" ""
+		(property "Footprint" "Teensy:GY-BNO08X_1x10_P2.54mm"
 			(at 107.95 147.32 0)
 			(hide yes)
@@
 			)
 		)
-		(property "Footprint" ""
+		(property "Footprint" "Teensy:Teensy41_PinNames"
 			(at 143.51 111.76 0)
 			(hide yes)

Commit message: add button
Parts:
- added R1: 10k Ω, Package_DIP:DIP-8_W7.62mm, symbol Device:R
- added SW2: SW_Push, Button_Switch_SMD:SW_SPST_CK_KMS2xxGP, symbol Switch:SW_Push
Connections:
- net at C1.2, C2.2, CS1.GND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: now also R1.1
- net at CS1.VIN (VIN_3.6_to_5.5_V), CS4.PMODE, D1.1 (K)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: now also SW2.2
- net at CS1.32: now also R1.2, SW2.1
- no-connect marks 45 -> 44
